File: PCB/robotArm.sch (KiCad schematic (older format))
At the start: 85 parts, among them J1 Motor_eje_X, J10 Gripper, J11 Conector Auxiliar 2, J12 5v, J13 End-Stop-X, J14 End-Stop-Y, J15 End-Stop-Z, J16 jumperLed5v, J17 Conector Auxiliar 1, J18 jumperLedVbat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

Commit message: PCB pull from master (#12)
* Update README.md

Se agregó descripción,  introducción y fuentes.

* Se consiguió una primera versión de Eje-Stop funcional

* Se inició una interfaz en python sencilla para la comunicación con el robot

* Se comenzó con conexión USB

* Se agregó LCD i2c y lógica de CDC

* update interface

* Se actualizaron los cambios

* return 2025

* El homming funciona!

* modo ejecución v1.0 funciona correctamente

* Se avanzo interfaz 3 modos funcionales v1.0

* actualizaciones en la interfaz

* Recuperando cambios del stash

* Se recuperaron las modificaciones de interfaz

* Se agregó leds en interfaz, botón de limpiar aprendizaje, se arregló configuración de velocidad en bluepill

* readme de stm32

* Se actualizo interfaz v1.0

* Se agregó rampa de velocidad

---------

Co-authored-by: Francisco Cano <100385537+FranciscoCano2@users.noreply.github.com>
Parts:
- removed C1: 103, Capacitor_THT:C_Disc_D8.0mm_W2.5mm_P5.00mm, symbol Device:C
- removed C6: 470uF, Capacitor_THT:CP_Radial_D8.0mm_P3.80mm, symbol Device:CP1
- removed D1, D13, D2, D3, D4, D5, D6, D7, D8, D9: 1N4007, Diode_THT:D_DO-41_SOD81_P10.16mm_Horizontal, symbol Diode:1N4007
- removed D12: LED_Vbat, LED_THT:LED_D5.0mm, symbol Device:LED
- removed J19: Vbat, TerminalBlock:TerminalBlock_bornier-2_P5.08mm, symbol Connector:Screw_Terminal_01x02
- removed R10: 220, Resistor_THT:R_Axial_DIN0207_L6.3mm_D2.5mm_P10.16mm_Horizontal, symbol Device:R_US
- added C19, C20: 103, Capacitor_THT:C_Disc_D8.0mm_W2.5mm_P5.00mm, symbol Device:C
- added D1: LED_Home, LED_THT:LED_D5.0mm, symbol Device:LED
- added D2: LED_Wait, LED_THT:LED_D5.0mm, symbol Device:LED
- added D3: LED_Finish, LED_THT:LED_D5.0mm, symbol Device:LED
- added R16, R17, R18: 1k, Resistor_THT:R_Axial_DIN0207_L6.3mm_D2.5mm_P10.16mm_Horizontal, symbol Device:R_US
- added R19: 10k, Resistor_THT:R_Axial_DIN0207_L6.3mm_D2.5mm_P10.16mm_Horizontal, symbol Device:R_US
- added SW2: STOP_EM, Button_Switch_THT:SW_PUSH_6mm_H5mm, symbol Switch:SW_Push
- C11, C8: value 470uF -> 10uF
- C5: value 47uF -> 10uF
- J18: value jumperLedVbat -> Pulsador Externo; footprint Connector_PinHeader_2.54mm:PinHeader_2x01_P2.54mm_Vertical -> Connector_PinHeader_2.54mm:PinHeader_1x02_P2.54mm_Vertical
- J5, J6, J7: footprint Connector_PinSocket_2.54mm:PinSocket_2x03_P2.54mm_Vertical -> Connector_PinHeader_2.54mm:PinHeader_2x03_P2.54mm_Vertical
- R12, R13, R7: value 10k -> 47k
- R2, R3, R4: value 10k -> 4.7k
- SW1: value SW_Push -> RESET
Connections:
- net labels added: STOP, finish, home, wait
- net labels removed: +BATT, ResetMotor, SleepMotor
- wire segments 485 -> 527
- no-connect marks 4 -> 5
Other:
- moved on the sheet: C10, C11, C12, C13, C14, C15, C16, C17, C18, C5, C7, C8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
